File: PCB/MixController.sch (KiCad schematic (older format))
At the start: 25 parts

Commit message: Create v0.0.7 schematic
Parts:
- removed J?: JST-SM2-FEMALE, symbol conn:Conn_01x02_Male
- removed J?: JST-SM2-MALE, symbol conn:Conn_01x02_Male
- removed J? (x2): Conn_01x02, symbol conn:Conn_01x02
- removed J?: Conn_01x07, symbol conn:Conn_01x07
- removed J? (x4): Conn_01x06, symbol conn:Conn_01x06
- removed J? (x2): Conn_01x04, symbol conn:Conn_01x04
- removed R?: 10K, symbol Device:R
- removed SW? (x3): SW_SPST, symbol switches:SW_SPST
- added J2: B2B-XH-A(LF)(SN), symbol conn:Conn_01x02_Male
- added J3: XHP-2, symbol conn:Conn_01x02_Female
- added J4, J8: XHP-3, symbol conn:Conn_01x03_Female
- added J7: B3B-XH-A(LF)(SN), symbol conn:Conn_01x03_Male
- added K1: G2R-1A-T DC48, symbol Relay:DIPxx-1Axx-11x
- added PS1: RSD-30H-24, symbol proj:RSD-30H-24
- added PS2: RSDW20H-05, symbol proj:RSDW20H-05
- added Q1: Q_NMOS_GDS, symbol Device:Q_NMOS_GDS
- added R2: 100K, symbol Device:R_Small
- added R3: 120, symbol Device:R
- added R4: 220, symbol Device:R
- added R5: 2.2K, symbol Device:R
- added SP1: LED_HOLDER_5MM, symbol proj:LED_HOLDER_5MM
- added SW1: Rotary_Selector_Switch, symbol proj:Rotary_Selector_Switch
- added U2: Adafruit_1096, symbol proj:Adafruit_1096
- added U3, U4: BOB-12009, symbol proj:BOB-12009
- added U5: GP2Y0A02YK0F, symbol proj:GP2Y0A02YK0F
- added U6: HSCDLNN001PDAA3, symbol proj:HSCDLNN001PDAA3
- D1: renamed from D?; MPN (none) -> C503B-GCS-CY0C0791; Vendor (none) -> DigiKey; Vendor P/N (none) -> C503B-GCS-CY0C0791-ND
- J1, J5, J6: renamed from J?; value Conn_01x02 -> PG7; MPN (none) -> a16101300ux0476; Vendor (none) -> Amazon; Vendor P/N (none) -> B01MSQI150
- J13, J14: renamed from J?; value Conn_01x08 -> PG7; MPN (none) -> a16101300ux0476; Vendor (none) -> Amazon; Vendor P/N (none) -> B01MSQI150
- R1: renamed from R?; Vendor (none) -> House
- SW5: renamed from SW?; value SW_SPST -> GRB136A05BB2; MPN (none) -> GRB136A05BB2; Vendor (none) -> DigiKey; Vendor P/N (none) -> SW652-ND
- SW6: renamed from SW?; MPN (none) -> PV1F240SS; Vendor (none) -> DigiKey; Vendor P/N (none) -> PV1F240SS-ND
- U1: renamed from U?; MPN (none) -> PHOTONH; Vendor (none) -> DigiKey; Vendor P/N (none) -> 1878-1000-ND
Connections:
- net labels added: +24V, +72V, PAIL_SNS, PRESS_SNS, PUMP_EN
- wire segments 160 -> 186
- no-connect marks 0 -> 15
Other:
- note added: "CABLE"
- note added: "Coil \nR: 4170K\nC: 11.5mA\nV: 48VDC"
- note added: "To Pump"
- note removed: "+5V"
- note removed: "1"
- note removed: "2"
- note removed: "3"
- note removed: "315Mhz Momentary"
- note removed: "4"
- note removed: "5"
- note removed: "6"
- note removed: "7"
- note removed: "8"
- note removed: "AURELIO TECH - B00QI6S68S"
- note removed: "BOB-12009"
- note removed: "D0"
- note removed: "D1"
- note removed: "D2"
- note removed: "D3"
- note removed: "DC/DC Converter \n(36-72V to 5V @1000mA)"
- note removed: "GND"
- note removed: "HV+"
- note removed: "HV1"
- note removed: "HV2"
- note removed: "HV3"
- note removed: "HV4"
- note removed: "LV+"
- note removed: "LV1"
- note removed: "LV2"
- note removed: "LV3"
- note removed: "LV4"
- note removed: "Level Translator"
- note removed: "NOTES:\nButton uses 3.3V source while motors use 5V source\nWire colors on motor side are best guess based on photos\nYou may want to use a 9 or 10 pin connector for Motor B to prevent them from being plugged incorrectly\nJST SM connectors picked for panel mount, swap with any connector available\nAll wire protrude 12" from box"
- note removed: "RF Reciever"
- note removed: "Rotary Selector Switch"
- note removed: "VIN+"
- note removed: "VIN-"
- note removed: "VT"
- note removed: "http://a.co/d/aNRq7J4"
- note removed: "https://www.adafruit.com/product/1096"
- note removed: "https://www.sparkfun.com/products/12009"

Commit message: Update connectors
Parts:
- added J10: B2B-XH-A(LF)(SN), symbol conn:Conn_01x02_Male
- added J11: B3B-XH-A(LF)(SN), symbol conn:Conn_01x03_Male
- added J12: XHP-3, symbol conn:Conn_01x03_Female
- added J9: XHP-2, symbol conn:Conn_01x02_Female
Connections:
- wire segments 186 -> 193

Commit message: Update
Other:
- note added: "14" Long\n8" Remove Sheath\nCut RED wire to 2""
- note added: "18" Long\n8" Remove Sheath\nCut BLACK wire to 2""
- note added: "18.5" Long\n12" Remove Sheath"
- note added: "22.5" Long\n12" Remove Sheath"
- note added: "HARDENER MOTOR POWER"
- note added: "RESIN MOTOR POWER"
- note removed: "18" Long\n5" Remove Sheath"
- note removed: "18" Long\n5" Remove Sheath\nCut BLACK wire to 2""
- note removed: "18" Long\n5" Remove Sheath\nCut RED wire to 2""
- note removed: "20" Long\n7" Remove Sheath"
- note removed: "MOTOR A POWER"
- note removed: "MOTOR B POWER"
Changed lines of the file:
@@
 $EndComp
 Text Notes 3650 2400 0    60   ~ 0
-MOTOR B POWER
+HARDENER MOTOR POWER
 Text Notes 3650 3100 0    60   ~ 0
-MOTOR A POWER
+RESIN MOTOR POWER
 Wire Wire Line
 	5150 4100 4900 4100
@@
 $EndComp
 Text Notes 9550 6150 0    60   ~ 0
-20" Long\n7" Remove Sheath
+22.5" Long\n12" Remove Sheath
 Text Label 7050 3650 0    60   ~ 0
 red
@@
 $EndComp
 Text Notes 9550 4300 0    60   ~ 0
-18" Long\n5" Remove Sheath
+18.5" Long\n12" Remove Sheath
 $Comp
 L conn:Conn_01x08 J13
@@
 Text Notes 10100 5850 0    39   ~ 0
 Same side as +VIN \n(RED)
-Text Notes 4500 2500 0    60   ~ 0
-18" Long\n5" Remove Sheath\nCut BLACK wire to 2"
-Text Notes 4500 3150 0    60   ~ 0
-18" Long\n5" Remove Sheath\nCut RED wire to 2"
+Text Notes 4950 2500 0    60   ~ 0
+18" Long\n8" Remove Sheath\nCut BLACK wire to 2"
+Text Notes 4950 3150 0    60   ~ 0
+14" Long\n8" Remove Sheath\nCut RED wire to 2"
 $Comp
 L switches:SW_SPST SW5

Commit message: Add 470 PD resistor to HV4 Inputs - Fix Pump Error
Parts:
- added R6, R7: 470, symbol Device:R_Small
Connections:
- wire segments 193 -> 199
Changed lines of the file:
@@
 	8800 5600 9350 5600
 Wire Wire Line
-	8900 5500 9350 5500
+	8900 5500 9050 5500
 Wire Wire Line
 	9000 5400 9350 5400
@@
 	8800 3750 9350 3750
 Wire Wire Line
-	8900 3650 9350 3650
+	8900 3650 9050 3650
 Wire Wire Line
 	9000 3550 9350 3550
@@
 Text Label 1700 5200 0    60   ~ 0
 white
+$Comp
+L Device:R_Small R7
+U 1 1 5BB04E7F
+P 9050 6000
+F 0 "R7" H 8991 5954 50  0000 R CNN
+F 1 "470" H 8991 6045 50  0000 R CNN
+F 2 "" H 9050 6000 50  0001 C CNN
+F 3 "~" H 9050 6000 50  0001 C CNN
+	1    9050 6000
+	-1   0    0    1
+$EndComp
+Wire Wire Line
+	9050 5900 9050 5500
+Connection ~ 9050 5500
+Wire Wire Line
+	9050 5500 9350 5500
+$Comp
+L power:GND #PWR035
+U 1 1 5BB10B21
+P 9050 6150
+F 0 "#PWR035" H 9050 5900 50  0001 C CNN
+F 1 "GND" H 9050 6000 50  0000 C CNN
+F 2 "" H 9050 6150 50  0001 C CNN
+F 3 "" H 9050 6150 50  0001 C CNN
+	1    9050 6150
+	1    0    0    -1
+$EndComp
+Wire Wire Line
+	9050 6150 9050 6100
+$Comp
+L Device:R_Small R6
+U 1 1 5BB1C9E8
+P 9050 4150
+F 0 "R6" H 8991 4104 50  0000 R CNN
+F 1 "470" H 8991 4195 50  0000 R CNN
+F 2 "" H 9050 4150 50  0001 C CNN
+F 3 "~" H 9050 4150 50  0001 C CNN
+	1    9050 4150
+	-1   0    0    1
+$EndComp
+Wire Wire Line
+	9050 4050 9050 3650
+Connection ~ 9050 3650
+Wire Wire Line
+	9050 3650 9350 3650
+$Comp
+L power:GND #PWR034
+U 1 1 5BB289F3
+P 9050 4300
+F 0 "#PWR034" H 9050 4050 50  0001 C CNN
+F 1 "GND" H 9050 4150 50  0000 C CNN
+F 2 "" H 9050 4300 50  0001 C CNN
+F 3 "" H 9050 4300 50  0001 C CNN
+	1    9050 4300
+	1    0    0    -1
+$EndComp
+Wire Wire Line
+	9050 4300 9050 4250
 $EndSCHEMATC

Commit message: Remove voltage divider on pail sensor output
Parts:
- removed R3: 120, symbol Device:R
- removed R4: 220, symbol Device:R
Connections:
- wire segments 199 -> 194
Changed lines of the file:
@@
 L proj:GP2Y0A02YK0F U5
 U 1 1 5BFBED5C
-P 1000 6250
-F 0 "U5" H 700 5950 60  0000 R CNN
-F 1 "GP2Y0A02YK0F" H 1250 6050 60  0000 R CNN
-F 2 "" H 850 6250 60  0001 C CNN
-F 3 "https://www.sparkfun.com/datasheets/Sensors/Infrared/gp2y0a02yk_e.pdf" H 850 6250 60  0001 C CNN
-F 4 "~" H 0   0   50  0001 C CNN "Alt Vendor"
-F 5 "~" H 0   0   50  0001 C CNN "Alt Vendor P/N"
-F 6 "GP2Y0A02YK0F" H 0   0   50  0001 C CNN "MPN"
-F 7 "SparkFun" H 0   0   50  0001 C CNN "Vendor"
-F 8 "SEN-08958" H 0   0   50  0001 C CNN "Vendor P/N"
-	1    1000 6250
+P 1300 6900
+F 0 "U5" H 1000 6600 60  0000 R CNN
+F 1 "GP2Y0A02YK0F" H 1550 6700 60  0000 R CNN
+F 2 "" H 1150 6900 60  0001 C CNN
+F 3 "https://www.sparkfun.com/datasheets/Sensors/Infrared/gp2y0a02yk_e.pdf" H 1150 6900 60  0001 C CNN
+F 4 "~" H 300 650 50  0001 C CNN "Alt Vendor"
+F 5 "~" H 300 650 50  0001 C CNN "Alt Vendor P/N"
+F 6 "GP2Y0A02YK0F" H 300 650 50  0001 C CNN "MPN"
+F 7 "SparkFun" H 300 650 50  0001 C CNN "Vendor"
+F 8 "SEN-08958" H 300 650 50  0001 C CNN "Vendor P/N"
+	1    1300 6900
 	1    0    0    1
 $EndComp
@@
 L power:+5V #PWR029
 U 1 1 5BFBF1CF
-P 2350 6050
-F 0 "#PWR029" H 2350 5900 50  0001 C CNN
-F 1 "+5V" H 2350 6190 50  0000 C CNN
-F 2 "" H 2350 6050 50  0001 C CNN
-F 3 "" H 2350 6050 50  0001 C CNN
-	1    2350 6050
-	1    0    0    -1
-$EndComp
-Wire Wire Line
-	2350 6050 2350 6150
-Wire Wire Line
-	2350 6150 2250 6150
+P 2650 6700
+F 0 "#PWR029" H 2650 6550 50  0001 C CNN
+F 1 "+5V" H 2650 6840 50  0000 C CNN
+F 2 "" H 2650 6700 50  0001 C CNN
+F 3 "" H 2650 6700 50  0001 C CNN
+	1    2650 6700
+	1    0    0    -1
+$EndComp
+Wire Wire Line
+	2650 6700 2650 6800
+Wire Wire Line
+	2650 6800 2550 6800
 $Comp
 L power:GND #PWR030
 U 1 1 5BFC822D
-P 2350 6600
-F 0 "#PWR030" H 2350 6350 50  0001 C CNN
-F 1 "GND" H 2350 6450 50  0000 C CNN
-F 2 "" H 2350 6600 50  0001 C CNN
-F 3 "" H 2350 6600 50  0001 C CNN
-	1    2350 6600
-	1    0    0    -1
-$EndComp
-$Comp
-L Device:R R3
-U 1 1 5BFDABB1
-P 2600 6500
-F 0 "R3" V 2700 6500 50  0000 C CNN
-F 1 "120" V 2600 6500 50  0000 C CNN
-F 2 "" V 2530 6500 50  0001 C CNN
-F 3 "" H 2600 6500 50  0001 C CNN
-F 4 "~" H -1750 1900 50  0001 C CNN "Alt Vendor"
-F 5 "~" H -1750 1900 50  0001 C CNN "Alt Vendor P/N"
-F 6 "~" H -1750 1900 50  0001 C CNN "MPN"
-F 7 "House" H -1750 1900 50  0001 C CNN "Vendor"
-F 8 "~" H -1750 1900 50  0001 C CNN "Vendor P/N"
-	1    2600 6500
-	-1   0    0    1
-$EndComp
-$Comp
-L Device:R R4
-U 1 1 5BFE4235
-P 2600 7050
-F 0 "R4" V 2700 7050 50  0000 C CNN
-F 1 "220" V 2600 7050 50  0000 C CNN
-F 2 "" V 2530 7050 50  0001 C CNN
-F 3 "" H 2600 7050 50  0001 C CNN
-F 4 "~" H -1750 2450 50  0001 C CNN "Alt Vendor"
-F 5 "~" H -1750 2450 50  0001 C CNN "Alt Vendor P/N"
-F 6 "~" H -1750 2450 50  0001 C CNN "MPN"
-F 7 "House" H -1750 2450 50  0001 C CNN "Vendor"
-F 8 "~" H -1750 2450 50  0001 C CNN "Vendor P/N"
-	1    2600 7050
-	-1   0    0    1
-$EndComp
-Wire Wire Line
-	2600 6650 2600 6800
-$Comp
-L power:GND #PWR031
-U 1 1 5BFED9FC
-P 2600 7350
-F 0 "#PWR031" H 2600 7100 50  0001 C CNN
-F 1 "GND" H 2600 7200 50  0000 C CNN
-F 2 "" H 2600 7350 50  0001 C CNN
-F 3 "" H 2600 7350 50  0001 C CNN
-	1    2600 7350
-	1    0    0    -1
-$EndComp
-Wire Wire Line
-	2600 7200 2600 7350
-Wire Wire Line
-	2600 6800 3150 6800
-Connection ~ 2600 6800
-Wire Wire Line
-	2600 6800 2600 6900
-Text Label 3150 6800 2    60   ~ 0
+P 2650 7250
+F 0 "#PWR030" H 2650 7000 50  0001 C CNN
+F 1 "GND" H 2650 7100 50  0000 C CNN
+F 2 "" H 2650 7250 50  0001 C CNN
+F 3 "" H 2650 7250 50  0001 C CNN
+	1    2650 7250
+	1    0    0    -1
+$EndComp
+Text Label 3150 6900 2    60   ~ 0
 PAIL_SNS
 Wire Wire Line
@@
 L conn:Conn_01x03_Female J4
 U 1 1 5C01523A
-P 1450 6250
-F 0 "J4" H 1400 6000 50  0000 L CNN
-F 1 "XHP-3" H 1350 5950 50  0001 L CNN
-F 2 "" H 1450 6250 50  0001 C CNN
-F 3 "http://www.jst-mfg.com/product/pdf/eng/eXH.pdf" H 1450 6250 50  0001 C CNN
-F 4 "~" H 0   0   50  0001 C CNN "Alt Vendor"
-F 5 "~" H 0   0   50  0001 C CNN "Alt Vendor P/N"
-F 6 "XHP-3" H 0   0   50  0001 C CNN "MPN"
-F 7 "DigiKey" H 0   0   50  0001 C CNN "Vendor"
-F 8 "455-2219-ND" H 0   0   50  0001 C CNN "Vendor P/N"
-	1    1450 6250
+P 1750 6900
+F 0 "J4" H 1700 6650 50  0000 L CNN
+F 1 "XHP-3" H 1650 6600 50  0001 L CNN
+F 2 "" H 1750 6900 50  0001 C CNN
+F 3 "http://www.jst-mfg.com/product/pdf/eng/eXH.pdf" H 1750 6900 50  0001 C CNN
+F 4 "~" H 300 650 50  0001 C CNN "Alt Vendor"
+F 5 "~" H 300 650 50  0001 C CNN "Alt Vendor P/N"
+F 6 "XHP-3" H 300 650 50  0001 C CNN "MPN"
+F 7 "DigiKey" H 300 650 50  0001 C CNN "Vendor"
+F 8 "455-2219-ND" H 300 650 50  0001 C CNN "Vendor P/N"
+	1    1750 6900
 	-1   0    0    1
 $EndComp
@@
 L conn:Conn_01x03_Male J7
 U 1 1 5C015301
-P 2050 6250
-F 0 "J7" H 2150 6500 50  0000 C CNN
-F 1 "B3B-XH-A(LF)(SN)" H 2000 6050 50  0001 C CNN
-F 2 "" H 2050 6250 50  0001 C CNN
-F 3 "http://www.jst-mfg.com/product/pdf/eng/eXH.pdf" H 2050 6250 50  0001 C CNN
-F 4 "~" H 0   0   50  0001 C CNN "Alt Vendor"
-F 5 "~" H 0   0   50  0001 C CNN "Alt Vendor P/N"
-F 6 "B3B-XH-A(LF)(SN)" H 0   0   50  0001 C CNN "MPN"
-F 7 "DigiKey" H 0   0   50  0001 C CNN "Vendor"
-F 8 "455-2248-ND" H 0   0   50  0001 C CNN "Vendor P/N"
-	1    2050 6250
+P 2350 6900
+F 0 "J7" H 2450 7150 50  0000 C CNN
+F 1 "B3B-XH-A(LF)(SN)" H 2300 6700 50  0001 C CNN
+F 2 "" H 2350 6900 50  0001 C CNN
+F 3 "http://www.jst-mfg.com/product/pdf/eng/eXH.pdf" H 2350 6900 50  0001 C CNN
+F 4 "~" H 300 650 50  0001 C CNN "Alt Vendor"
+F 5 "~" H 300 650 50  0001 C CNN "Alt Vendor P/N"
+F 6 "B3B-XH-A(LF)(SN)" H 300 650 50  0001 C CNN "MPN"
+F 7 "DigiKey" H 300 650 50  0001 C CNN "Vendor"
+F 8 "455-2248-ND" H 300 650 50  0001 C CNN "Vendor P/N"
+	1    2350 6900
 	1    0    0    -1
 $EndComp
@@
 L conn:Conn_01x03_Female J8
 U 1 1 5C029783
-P 2050 6250
-F 0 "J8" H 1950 6500 50  0000 L CNN
-F 1 "XHP-3" H 1850 6600 50  0001 L CNN
-F 2 "" H 2050 6250 50  0001 C CNN
-F 3 "http://www.jst-mfg.com/product/pdf/eng/eXH.pdf" H 2050 6250 50  0001 C CNN
-F 4 "~" H 0   0   50  0001 C CNN "Alt Vendor"
-F 5 "~" H 0   0   50  0001 C CNN "Alt Vendor P/N"
-F 6 "XHP-3" H 0   0   50  0001 C CNN "MPN"
-F 7 "DigiKey" H 0   0   50  0001 C CNN "Vendor"
-F 8 "455-2219-ND" H 0   0   50  0001 C CNN "Vendor P/N"
-	1    2050 6250
-	1    0    0    -1
-$EndComp
-Wire Wire Line
-	1650 6150 1850 6150
-Wire Wire Line
-	1650 6250 1850 6250
-Wire Wire Line
-	1650 6350 1850 6350
-Wire Notes Line
-	1550 6050 1550 6400
-Wire Notes Line
-	1550 6400 1950 6400
-Wire Notes Line
-	1950 6400 1950 6050
-Wire Notes Line
-	1950 6050 1550 6050
-Text Notes 1600 6050 0    60   ~ 0
+P 2350 6900
+F 0 "J8" H 2250 7150 50  0000 L CNN
+F 1 "XHP-3" H 2150 7250 50  0001 L CNN
+F 2 "" H 2350 6900 50  0001 C CNN
+F 3 "http://www.jst-mfg.com/product/pdf/eng/eXH.pdf" H 2350 6900 50  0001 C CNN
+F 4 "~" H 300 650 50  0001 C CNN "Alt Vendor"
+F 5 "~" H 300 650 50  0001 C CNN "Alt Vendor P/N"
+F 6 "XHP-3" H 300 650 50  0001 C CNN "MPN"
+F 7 "DigiKey" H 300 650 50  0001 C CNN "Vendor"
+F 8 "455-2219-ND" H 300 650 50  0001 C CNN "Vendor P/N"
+	1    2350 6900
+	1    0    0    -1
+$EndComp
+Wire Wire Line
+	1950 6800 2150 6800
+Wire Wire Line
+	1950 6900 2150 6900
+Wire Wire Line
+	1950 7000 2150 7000
+Wire Notes Line
+	1850 6700 1850 7050
+Wire Notes Line
+	1850 7050 2250 7050
+Wire Notes Line
+	2250 7050 2250 6700
+Wire Notes Line
+	2250 6700 1850 6700
+Text Notes 1900 6700 0    60   ~ 0
 CABLE
 $Comp
@@
 Text Notes 2100 2200 0    60   ~ 0
 Coil \nR: 4170K\nC: 11.5mA\nV: 48VDC
-NoConn ~ 1450 6150
-NoConn ~ 1450 6250
-NoConn ~ 1450 6350
+NoConn ~ 1750 6800
+NoConn ~ 1750 6900
+NoConn ~ 1750 7000
 $Comp
 L proj:+72V #PWR0101
@@
 Connection ~ 2550 5650
 Wire Wire Line
-	2250 6350 2350 6350
-Wire Wire Line
-	2350 6350 2350 6600
-Wire Wire Line
-	2250 6250 2600 6250
-Wire Wire Line
-	2600 6250 2600 6350
-Text Label 1700 6150 0    60   ~ 0
+	2550 7000 2650 7000
+Wire Wire Line
+	2650 7000 2650 7250
+Wire Wire Line
+	2550 6900 3150 6900
+Text Label 2000 6800 0    60   ~ 0
 red
-Text Label 1650 6350 0    60   ~ 0
+Text Label 1950 7000 0    60   ~ 0
 black
-Text Label 1650 6250 0    60   ~ 0
+Text Label 1950 6900 0    60   ~ 0
 white
 Text Label 1750 5550 0    60   ~ 0

Commit message: Add I/O and ADC Expanders
Parts:
- removed D1: LED, symbol Device:LED
- removed J10: B2B-XH-A(LF)(SN), symbol conn:Conn_01x02_Male
- removed J11: B3B-XH-A(LF)(SN), symbol conn:Conn_01x03_Male
- removed J12: XHP-3, symbol conn:Conn_01x03_Female
- removed J9: XHP-2, symbol conn:Conn_01x02_Female
- added D1: LED_CRGB, symbol Device:LED_CRGB
- added J10: XHP-2, symbol conn:Conn_01x02_Female
- added J11: Conn_01x05_Male, symbol Connector:Conn_01x05_Male
- added J12: Conn_01x05_Female, symbol Connector:Conn_01x05_Female
- added J15, J16, J17, J18, J19, J20, J21, J22, J23, J24, J25, J26, J27, J28, J29, J30, J31, J32, J33, J34, J35, J36, J37, J38, J39, J40, J41, J42, J43, J44, J45, J46, J47, J48, J49, J50, J51, J52, J53, J54, J55, J56, J57, J58, J59, J60, J61, J62, J63, J64, J65, J66, J67, J68, J69, J70, J71, J72, J73, J74, J75, J76, J77, J78, J79, J80, J81, J82, J83, J84, J85, J86, J87, J88, J89, J90: TEST_1P, symbol conn:TEST_1P
- added J9: B2B-XH-A(LF)(SN), symbol conn:Conn_01x02_Male
- added J91: Conn_01x04_Male, symbol Connector:Conn_01x04_Male
- added J92: Conn_01x04_Female, symbol Connector:Conn_01x04_Female
- added JP1, JP10, JP11, JP12, JP13, JP14, JP15, JP16, JP17, JP18, JP19, JP2, JP20, JP21, JP22, JP23, JP3, JP4, JP5, JP6, JP7, JP8, JP9: Jumper_NC_Small, symbol Device:Jumper_NC_Small
- added R3, R4: 4.7K, symbol Device:R_Small
- added R8, R9: 330, symbol Device:R
- added U7: MCP23017, symbol microchip:MCP23017
- added U8: ADS7830, Package_SO:TSSOP-16_4.4x5mm_P0.65mm, symbol Analog_DAC:ADS7830
Connections:
- net labels added: HARDENER_ENABLE, HARDENER_HLFB, HARDENER_INPUT_A, HARDENER_INPUT_B, LIQUID_SENSE, RESIN_ENABLE, RESIN_HLFB, RESIN_INPUT_A, RESIN_INPUT_B, ROTARY_1, ROTARY_2, ROTARY_3, ROTARY_4, SCL, SDA, STATUS_LED_B, STATUS_LED_G, STATUS_LED_R, USER_BUTTON, USER_REMOTE
- net labels removed: green
- wire segments 194 -> 404
- no-connect marks 15 -> 14
Other:
- note added: "Black"
- note added: "Blue"
- note added: "Green"
- note added: "HARDENER PUMP"
- note added: "RESIN PUMP"
- note added: "Red"
- note added: "White"
- note added: "Yellow"
- note removed: "To Motor A"
- note removed: "To Motor B"

Commit message: Add footprints, Add connector between cable power and board
Parts:
- removed J14: PG7, symbol conn:Conn_01x08
- removed PS1: RSD-30H-24, symbol proj:RSD-30H-24
- added J14, J96: XHP-8, symbol Connector:Conn_01x08_Female
- added J93: 50-57-9402, ~, symbol conn:Conn_01x02_Female
- added J94: 0705430001, Connectors_Molex:Molex_SPOX-5267_22-03-5025_02x2.54mm_Straight, symbol conn:Conn_01x02_Male
- added J95: B8B-XH-A(LF)(SN), Connectors_JST:JST_XH_B08B-XH-A_08x2.50mm_Straight, symbol Connector:Conn_01x08_Male
- added PS1: TMR_6-7215WIR, local:TRACO_TMR_6, symbol proj:TMR_6-7215WIR
- added SP2, SP3, SP4, SP5, SP6, SP7: PG7, ~, symbol proj:PG7
- D1: footprint (none) -> ~; Vendor (none) -> DigiKey
- J1, J10, J3, J4, J5, J6, J8, K1, R5, SP1, SW1, SW5, U5: footprint (none) -> ~
- J11: value Conn_01x05_Male -> B5B-XH-A(LF)(SN); footprint (none) -> Connectors_JST:JST_XH_B05B-XH-A_05x2.50mm_Straight; MPN (none) -> B5B-XH-A(LF)(SN); Vendor (none) -> DigiKey; Vendor P/N (none) -> 455-2270-ND
- J12: value Conn_01x05_Female -> XHP-5; footprint (none) -> ~; MPN (none) -> XHP-5; Vendor (none) -> DigiKey; Vendor P/N (none) -> 455-2268-ND
- J13: value PG7 -> B8B-XH-A(LF)(SN); footprint (none) -> Connectors_JST:JST_XH_B08B-XH-A_08x2.50mm_Straight; symbol conn:Conn_01x08 -> Connector:Conn_01x08_Male; MPN a16101300ux0476 -> B8B-XH-A(LF)(SN); Vendor Amazon -> DigiKey; Vendor P/N B01MSQI150 -> 455-2251-ND
- J15, J16, J17, J18, J19, J20, J21, J22, J23, J24, J25, J26, J27, J28, J29, J30, J31, J32, J33, J34, J35, J36, J37, J38, J39, J40, J41, J42, J43, J44, J45, J46, J47, J48, J49, J50, J51, J52, J53, J54, J55, J56, J57, J58, J59, J60, J61, J62, J63, J64, J65, J66, J67, J68, J69, J70, J71, J72, J73, J74, J75, J76, J77, J78, J79, J80, J81, J82, J83, J84, J85, J86, J87, J88, J89, J90: value TEST_1P -> ~; footprint (none) -> local:SinglePinHeader2.54Pitch
- J2, J9: footprint (none) -> Connectors_JST:JST_XH_B02B-XH-A_05x2.50mm_Straight
- J7: footprint (none) -> Connectors_JST:JST_XH_B03B-XH-A_05x2.50mm_Straight
- J91: value Conn_01x04_Male -> B4B-XH-A(LF)(SN); footprint (none) -> Connectors_JST:JST_XH_B04B-XH-A_05x2.50mm_Straight; MPN (none) -> B4B-XH-A(LF)(SN); Vendor (none) -> DigiKey; Vendor P/N (none) -> 455-2249-ND
- J92: value Conn_01x04_Female -> XHP-4; footprint (none) -> ~; MPN (none) -> XHP-4; Vendor (none) -> DigiKey; Vendor P/N (none) -> 455-2267-ND
- JP1, JP10, JP11, JP12, JP13, JP14, JP15, JP16, JP17, JP18, JP19, JP2, JP20, JP21, JP22, JP23, JP3, JP4, JP5, JP6, JP7, JP8, JP9: footprint (none) -> Jumper:SolderJumper-2_P1.3mm_Open_RoundedPad1.0x1.5mm
- PS2: footprint (none) -> local:RSDW20_H
- Q1: footprint (none) -> TO_SOT_Packages_THT:TO-220-3_Horizontal
- R1, R2, R8, R9: footprint (none) -> Resistors_THT:R_Axial_DIN0207_L6.3mm_D2.5mm_P10.16mm_Horizontal
- R3, R4, R6, R7: footprint (none) -> Resistors_THT:R_Axial_DIN0207_L6.3mm_D2.5mm_P10.16mm_Horizontal; Vendor (none) -> House
- SW6: value SW_Push -> PV1F240SS; footprint (none) -> ~
- U1: footprint (none) -> Particle:photon_smd
- U2: footprint (none) -> local:Adafruit_1096
- U3, U4: footprint (none) -> Housings_DIP:DIP-12_W10.16mm
- U6: footprint (none) -> local:HoneyWell_LN
- U7: footprint (none) -> Housings_DIP:DIP-28_W7.62mm
Connections:
- wire segments 404 -> 450
- no-connect marks 14 -> 16
