File: PCB/MixController.sch (KiCad schematic (older format))
At the start: 151 parts, among them J1 PG7, J10 XHP-2, J11 B5B-XH-A(LF)(SN), J12 XHP-5, J13 B8B-XH-A(LF)(SN), J14 XHP-8, J2 B2B-XH-A(LF)(SN), J3 XHP-2, J4 XHP-3, J5 PG7, J6 PG7, J7 B3B-XH-A(LF)(SN), J8 XHP-3, J9 B2B-XH-A(LF)(SN), J91 B4B-XH-A(LF)(SN), J92 XHP-4, J93 50-57-9402, J94 0705430001, J95 B8B-XH-A(LF)(SN), J96 XHP-8, K1 G2R-1A-T DC48, Q1 Q_NMOS_GDS, SW1 Rotary_Selector_Switch, SW5 GRB136A05BB2, SW6 PV1F240SS, U1 PARTICLE_PHOTON, U2 Adafruit_1096, U3 BOB-12009, U4 BOB-12009, U5 GP2Y0A02YK0F, U6 HSCDLNN001PDAA3, U7 MCP23017, U8 ADS7830

Commit message: Start Layout
Parts:
- removed U1: PARTICLE_PHOTON, Particle:photon_smd, symbol particle:PARTICLE_PHOTON
- added J97: B4B-PH-K-S(LF)(SN), Connector_JST:JST_PH_B4B-PH-K_1x04_P2.00mm_Vertical, symbol Connector:Conn_01x04_Male
- added J98: 455-1164-ND, ~, symbol Connector:Conn_01x04_Female
- added J99: USB_B, ~, symbol Connector:USB_B
- added U1: Photon, Particle:photon_smd, symbol MCU_Particle:Photon
- J11: footprint Connectors_JST:JST_XH_B05B-XH-A_05x2.50mm_Straight -> Connector_JST:JST_XH_B05B-XH-A_1x05_P2.50mm_Vertical
- J13, J95: footprint Connectors_JST:JST_XH_B08B-XH-A_08x2.50mm_Straight -> Connector_JST:JST_XH_B08B-XH-A_1x08_P2.50mm_Vertical
- J14, J96: footprint (none) -> ~
- J15, J16, J17, J18, J19, J20, J21, J22, J23, J24, J25, J26, J27, J28, J29, J30, J31, J32, J33, J34, J35, J36, J37, J38, J39, J40, J41, J42, J43, J44, J45, J46, J47, J48, J49, J50, J51, J52, J53, J54, J55, J56, J57, J58, J59, J60, J61, J62, J63, J64, J65, J66, J67, J68, J69, J70, J71, J72, J73, J74, J75, J76, J77, J78, J79, J80, J81, J82, J83, J84, J85, J86, J87, J88, J89, J90: footprint local:SinglePinHeader2.54Pitch -> Local:ConnectorPoint_THT_D1.5mm_Drill-0.7mm
- J2, J9: footprint Connectors_JST:JST_XH_B02B-XH-A_05x2.50mm_Straight -> Connector_JST:JST_XH_B02B-XH-A_1x02_P2.50mm_Vertical
- J7: footprint Connectors_JST:JST_XH_B03B-XH-A_05x2.50mm_Straight -> Connector_JST:JST_XH_B03B-XH-A_1x03_P2.50mm_Vertical
- J91: footprint Connectors_JST:JST_XH_B04B-XH-A_05x2.50mm_Straight -> Connector_JST:JST_XH_B04B-XH-A_1x04_P2.50mm_Vertical
- J94: footprint Connectors_Molex:Molex_SPOX-5267_22-03-5025_02x2.54mm_Straight -> Connector_Molex:Molex_SPOX_5267-02A_1x02_P2.50mm_Vertical
- JP1, JP10, JP11, JP12, JP13, JP14, JP15, JP16, JP17, JP18, JP19, JP2, JP20, JP21, JP22, JP23, JP3, JP4, JP5, JP6, JP7, JP8, JP9: value Jumper_NC_Small -> ~
- PS1: footprint local:TRACO_TMR_6 -> (none)
- PS2: footprint local:RSDW20_H -> (none)
- Q1: footprint TO_SOT_Packages_THT:TO-220-3_Horizontal -> Package_TO_SOT_THT:TO-220-3_Horizontal_TabDown
- R1, R8, R9: value 330 -> 470; footprint Resistors_THT:R_Axial_DIN0207_L6.3mm_D2.5mm_P10.16mm_Horizontal -> Resistor_THT:R_Axial_DIN0207_L6.3mm_D2.5mm_P10.16mm_Horizontal
- R2, R3, R4: footprint Resistors_THT:R_Axial_DIN0207_L6.3mm_D2.5mm_P10.16mm_Horizontal -> Resistor_THT:R_Axial_DIN0207_L6.3mm_D2.5mm_P10.16mm_Horizontal
- R6, R7: value 470 -> 1K; footprint Resistors_THT:R_Axial_DIN0207_L6.3mm_D2.5mm_P10.16mm_Horizontal -> Resistor_THT:R_Axial_DIN0207_L6.3mm_D2.5mm_P10.16mm_Horizontal
- U2: footprint local:Adafruit_1096 -> (none)
- U3, U4: footprint Housings_DIP:DIP-12_W10.16mm -> (none)
- U6: footprint local:HoneyWell_LN -> (none)
- U7: footprint Housings_DIP:DIP-28_W7.62mm -> Package_DIP:DIP-28_W7.62mm
Connections:
- net labels added: USB(+), USB(-)
- wire segments 450 -> 478
- no-connect marks 16 -> 18
