File: PCB/MixController.sch (KiCad schematic (older format))
At the start: 154 parts, among them J1 PG7, J10 XHP-2, J11 B5B-XH-A(LF)(SN), J12 XHP-5, J13 B8B-XH-A(LF)(SN), J14 XHP-8, J2 B2B-XH-A(LF)(SN), J3 XHP-2, J4 XHP-3, J5 PG7, J6 PG7, J7 B3B-XH-A(LF)(SN), J8 XHP-3, J9 B2B-XH-A(LF)(SN), J91 B4B-XH-A(LF)(SN), J92 XHP-4, J93 50-57-9402, J94 0705430001, J95 B8B-XH-A(LF)(SN), J96 XHP-8, J97 B4B-PH-K-S(LF)(SN), J98 455-1164-ND, J99 USB_B, K1 G2R-1A-T DC48, Q1 Q_NMOS_GDS, SW1 Rotary_Selector_Switch, SW5 GRB136A05BB2, SW6 PV1F240SS, U1 Photon, U2 Adafruit_1096, U3 BOB-12009, U4 BOB-12009, U5 GP2Y0A02YK0F, U6 HSCDLNN001PDAA3, U7 MCP23017, U8 ADS7830

Commit message: Update Libraries
Parts:
- J1, J5, J6: symbol conn:Conn_01x02 -> Connector:Conn_01x02_Female
- J10, J3, J93: symbol conn:Conn_01x02_Female -> Connector:Conn_01x02_Female
- J15, J16, J17, J18, J19, J20, J21, J22, J23, J24, J25, J26, J27, J28, J29, J30, J31, J32, J33, J34, J35, J36, J37, J38, J39, J40, J41, J42, J43, J44, J45, J46, J47, J48, J49, J50, J51, J52, J53, J54, J55, J56, J57, J58, J59, J60, J61, J62, J63, J64, J65, J66, J67, J68, J69, J70, J71, J72, J73, J74, J75, J76, J77, J78, J79, J80, J81, J82, J83, J84, J85, J86, J87, J88, J89, J90: symbol conn:TEST_1P -> Connector:TestPoint
- J2, J9, J94: symbol conn:Conn_01x02_Male -> Connector:Conn_01x02_Male
- J4, J8: symbol conn:Conn_01x03_Female -> Connector:Conn_01x03_Female
- J7: symbol conn:Conn_01x03_Male -> Connector:Conn_01x03_Male
- PS1: symbol proj:TMR_6-7215WIR -> VDW_Modules:TMR_6-7215WIR
- PS2: symbol proj:RSDW20H-05 -> VDW_Modules:RSDW20H-05
- SP1: symbol proj:LED_HOLDER_5MM -> VDW_Mechanical:LED_HOLDER_5MM
- SP2, SP3, SP4, SP5, SP6, SP7: symbol proj:PG7 -> VDW_Mechanical:PG7
- SW1: symbol proj:Rotary_Selector_Switch -> VDW_Modules:Rotary_Selector_Switch
- SW5: symbol switches:SW_SPST -> Switch:SW_SPST
- SW6: symbol switches:SW_Push -> Switch:SW_Push
- U1: symbol MCU_Particle:Photon -> MCU_Particle-VDW:Photon
- U2: symbol proj:Adafruit_1096 -> VDW_Modules:Adafruit_1096
- U3, U4: symbol proj:BOB-12009 -> VDW_Modules:BOB-12009
- U5: symbol proj:GP2Y0A02YK0F -> VDW_Modules:GP2Y0A02YK0F
- U6: symbol proj:HSCDLNN001PDAA3 -> VDW_Modules:HSCDLNN001PDAA3
- U7: symbol microchip:MCP23017 -> Interface_Expansion:MCP23017_SP

Commit message: Add temporary voltage divider
Other:
- note added: "Temporarily SSCDRRN005PGAA5\nwith 2.2K and 4.7K voltage divider"
Changed lines of the file:
@@
 Text Notes 1200 5300 0    60   ~ 0
 KNOB: ML-75-1-6
+Text Notes 1550 8950 0    60   ~ 0
+Temporarily SSCDRRN005PGAA5\nwith 2.2K and 4.7K voltage divider
 $EndSCHEMATC

Commit message: Add indicator leds, chime speaker, update layout
Parts:
- added D2: +72V, symbol Device:LED_ALT
- added D3: +5V, symbol Device:LED_ALT
- added D4: +24V, symbol Device:LED_ALT
- added D5: EN_HARD, symbol Device:LED_ALT
- added D6: EN_RESIN, symbol Device:LED_ALT
- added D7: PUMP, symbol Device:LED_ALT
- added J100: PHR-2, ~, symbol Connector:Conn_01x02_Female
- added J101: B2B-PH-K-S(LF)(SN), Connector_JST:JST_PH_B2B-PH-K_1x02_P2.00mm_Vertical, symbol Connector:Conn_01x02_Male
- added J102: PHR-3, ~, symbol Connector:Conn_01x03_Female
- added J103: B3B-PH-K-S(LF)(SN), Connector_JST:JST_PH_B3B-PH-K_1x03_P2.00mm_Vertical, symbol Connector:Conn_01x03_Male
- added J104: B2B-XH-A(LF)(SN), Connector_JST:JST_XH_B02B-XH-A_1x02_P2.50mm_Vertical, symbol Connector:Conn_01x02_Male
- added J105: XHP-2, ~, symbol Connector:Conn_01x02_Female
- added JP24, JP25, JP26: ~, Jumper:SolderJumper-2_P1.3mm_Open_RoundedPad1.0x1.5mm, symbol Device:Jumper_NC_Small
- added LS1: Speaker, symbol Device:Speaker
- added Q2: Q_NMOS_GDS, Package_TO_SOT_THT:TO-220-3_Horizontal_TabDown, symbol Device:Q_NMOS_GDS
- added R10, R11: 10K .01%, Resistor_SMD:R_0805_2012Metric_Pad1.15x1.40mm_HandSolder, symbol Device:R_Small
- added R12: 23k, symbol Device:R_Small
- added R13, R16, R17: 1k, symbol Device:R_Small
- added R14, R18: 7k, symbol Device:R_Small
- added R15: 100K, Resistor_THT:R_Axial_DIN0207_L6.3mm_D2.5mm_P10.16mm_Horizontal, symbol Device:R_Small
- added TH1, TH2: 10K, symbol Device:Thermistor
- added TP1: SCL, TestPoint:TestPoint_THTPad_D1.5mm_Drill0.7mm, symbol Connector:TestPoint
- added TP2: SDA, TestPoint:TestPoint_THTPad_D1.5mm_Drill0.7mm, symbol Connector:TestPoint
- D1: value LED_CRGB -> LED_ARGB; symbol Device:LED_CRGB -> Device:LED_ARGB
- U7: value MCP23017 -> MCP23017_SP
Connections:
- net labels added: CHIME, THERM_HARDENER, THERM_RESIN
- wire segments 478 -> 557
- no-connect marks 18 -> 28
Other:
- note removed: "Black"

Commit message: update schematic per ECN Maxx 5
Parts:
- removed J38, J55, J67, J71: ~, Local:ConnectorPoint_THT_D1.5mm_Drill-0.7mm, symbol Connector:TestPoint
- added C1, C2, C3, C4: 0.1u, Capacitor_SMD:C_0805_2012Metric_Pad1.15x1.40mm_HandSolder, symbol Device:C_Small
- added C5: 470u, Capacitor_SMD:C_0805_2012Metric_Pad1.15x1.40mm_HandSolder, symbol Device:C_Small
- added D10: STEP_HARD, LED_SMD:LED_0805_2012Metric_Pad1.15x1.40mm_HandSolder, symbol Device:LED_ALT
- added D11: STEP_RESIN, LED_SMD:LED_0805_2012Metric_Pad1.15x1.40mm_HandSolder, symbol Device:LED_ALT
- added D8: LIQ_RESIN, LED_SMD:LED_0805_2012Metric_Pad1.15x1.40mm_HandSolder, symbol Device:LED_ALT
- added D9: LIQ_HARD, LED_SMD:LED_0805_2012Metric_Pad1.15x1.40mm_HandSolder, symbol Device:LED_ALT
- added J38: B5B-PH-K-S(LF)(SN), Connector_JST:JST_PH_B5B-PH-K_1x05_P2.00mm_Vertical, symbol Connector:Conn_01x05_Male
- added J55: PHR-5, ~, symbol Connector:Conn_01x05_Female
- added J67: B6B-PH-K-S(LF)(SN), Connector_JST:JST_PH_B6B-PH-K_1x06_P2.00mm_Vertical, symbol Connector:Conn_01x06_Male
- added J71: PHR-6, ~, symbol Connector:Conn_01x06_Female
- added JP27: ~, Jumper:SolderJumper-2_P1.3mm_Open_RoundedPad1.0x1.5mm, symbol Device:Jumper_NC_Small
- added R19, R20: 10k, Resistor_SMD:R_0805_2012Metric_Pad1.15x1.40mm_HandSolder, symbol Device:R_Small
- added R21, R22: 470, Resistor_SMD:R_0805_2012Metric_Pad1.15x1.40mm_HandSolder, symbol Device:R_Small
- added R23, R24: 1k, Resistor_SMD:R_0805_2012Metric_Pad1.15x1.40mm_HandSolder, symbol Device:R_Small
- added U10, U9: FL50, ~, symbol Relay:DIPxx-1Cxx-51x
- D2, D3, D4, D5, D6, D7: footprint (none) -> LED_SMD:LED_0805_2012Metric_Pad1.15x1.40mm_HandSolder
- J98: value 455-1164-ND -> PHR-4
- LS1, TH1, TH2: footprint (none) -> ~
- R10, R11: value 10K .01% -> 5K .01%
- R12, R13, R14, R16, R17, R18: footprint (none) -> Resistor_SMD:R_0805_2012Metric_Pad1.15x1.40mm_HandSolder
- R15, R2: footprint Resistor_THT:R_Axial_DIN0207_L6.3mm_D2.5mm_P10.16mm_Horizontal -> Resistor_SMD:R_0805_2012Metric_Pad1.15x1.40mm_HandSolder
Connections:
- net labels added: HARDENER_INPUT_DIR, HARDENER_INPUT_STEP, LIQUID_SNS_HARDENER, LIQUID_SNS_RESIN, RESIN_INPUT_DIR, RESIN_INPUT_STEP
- net labels removed: HARDENER_INPUT_A, HARDENER_INPUT_B, LIQUID_SENSE, RESIN_INPUT_A, RESIN_INPUT_B, black, red, white
- wire segments 557 -> 637
- no-connect marks 28 -> 36
Other:
- note added: "Black"

Commit message: Update Layout
Parts:
- R1, R3, R4, R6, R7, R8, R9: footprint Resistor_THT:R_Axial_DIN0207_L6.3mm_D2.5mm_P10.16mm_Horizontal -> Resistor_SMD:R_0805_2012Metric_Pad1.15x1.40mm_HandSolder
Other:
- note added: "84V When Charging"
Changed lines of the file:
@@
 F 0 "R1" V 13500 8250 50  0000 C CNN
 F 1 "470" V 13400 8250 50  0000 C CNN
-F 2 "Resistor_THT:R_Axial_DIN0207_L6.3mm_D2.5mm_P10.16mm_Horizontal" V 13330 8250 50  0001 C CNN
+F 2 "Resistor_SMD:R_0805_2012Metric_Pad1.15x1.40mm_HandSolder" V 13330 8250 50  0001 C CNN
 F 3 "~" H 13400 8250 50  0001 C CNN
 F 4 "~" H 9050 3650 50  0001 C CNN "Alt Vendor"
@@
 	13700 4350 14350 4350
 Wire Wire Line
-	13700 4250 14350 4250
+	13700 4250 13900 4250
 Wire Wire Line
 	14000 4050 14350 4050
@@
 Text Label 14450 1400 0    60   ~ 0
 PUMP_EN
-Text Label 7350 5500 0    60   ~ 0
+Text Label 7350 5700 0    60   ~ 0
 PUMP_EN
 Text Label 7450 3150 0    60   ~ 0
@@
 F 0 "R7" H 13541 7004 50  0000 R CNN
 F 1 "1K" H 13541 7095 50  0000 R CNN
-F 2 "Resistor_THT:R_Axial_DIN0207_L6.3mm_D2.5mm_P10.16mm_Horizontal" H 13600 7050 50  0001 C CNN
+F 2 "Resistor_SMD:R_0805_2012Metric_Pad1.15x1.40mm_HandSolder" H 13600 7050 50  0001 C CNN
 F 3 "~" H 13600 7050 50  0001 C CNN
 F 4 "~" H -450 1500 50  0001 C CNN "Alt Vendor"
@@
 F 0 "R6" H 13541 4654 50  0000 R CNN
 F 1 "1K" H 13541 4745 50  0000 R CNN
-F 2 "Resistor_THT:R_Axial_DIN0207_L6.3mm_D2.5mm_P10.16mm_Horizontal" H 13600 4700 50  0001 C CNN
+F 2 "Resistor_SMD:R_0805_2012Metric_Pad1.15x1.40mm_HandSolder" H 13600 4700 50  0001 C CNN
 F 3 "~" H 13600 4700 50  0001 C CNN
 F 4 "~" H -450 950 50  0001 C CNN "Alt Vendor"
@@
 F 0 "R3" H 9159 9246 50  0000 L CNN
 F 1 "4.7K" H 9159 9155 50  0000 L CNN
-F 2 "Resistor_THT:R_Axial_DIN0207_L6.3mm_D2.5mm_P10.16mm_Horizontal" H 9100 9200 50  0001 C CNN
+F 2 "Resistor_SMD:R_0805_2012Metric_Pad1.15x1.40mm_HandSolder" H 9100 9200 50  0001 C CNN
 F 3 "~" H 9100 9200 50  0001 C CNN
 F 4 "~" H -100 1050 50  0001 C CNN "Alt Vendor"
@@
 F 0 "R4" H 9509 9246 50  0000 L CNN
 F 1 "4.7K" H 9509 9155 50  0000 L CNN
-F 2 "Resistor_THT:R_Axial_DIN0207_L6.3mm_D2.5mm_P10.16mm_Horizontal" H 9450 9200 50  0001 C CNN
+F 2 "Resistor_SMD:R_0805_2012Metric_Pad1.15x1.40mm_HandSolder" H 9450 9200 50  0001 C CNN
 F 3 "~" H 9450 9200 50  0001 C CNN
 F 4 "~" H -100 1050 50  0001 C CNN "Alt Vendor"
@@
 F 0 "R8" V 13500 8450 50  0000 C CNN
 F 1 "470" V 13400 8450 50  0000 C CNN
-F 2 "Resistor_THT:R_Axial_DIN0207_L6.3mm_D2.5mm_P10.16mm_Horizontal" V 13330 8450 50  0001 C CNN
+F 2 "Resistor_SMD:R_0805_2012Metric_Pad1.15x1.40mm_HandSolder" V 13330 8450 50  0001 C CNN
 F 3 "~" H 13400 8450 50  0001 C CNN
 F 4 "~" H 9050 3850 50  0001 C CNN "Alt Vendor"
@@
 F 0 "R9" V 13500 8650 50  0000 C CNN
 F 1 "470" V 13400 8650 50  0000 C CNN
-F 2 "Resistor_THT:R_Axial_DIN0207_L6.3mm_D2.5mm_P10.16mm_Horizontal" V 13330 8650 50  0001 C CNN
+F 2 "Resistor_SMD:R_0805_2012Metric_Pad1.15x1.40mm_HandSolder" V 13330 8650 50  0001 C CNN
 F 3 "~" H 13400 8650 50  0001 C CNN
 F 4 "~" H 9050 4050 50  0001 C CNN "Alt Vendor"
@@
 Wire Wire Line
 	8350 5700 7350 5700
-Text Label 7350 5700 0    60   ~ 0
+Text Label 7350 5500 0    60   ~ 0
 LIQUID_SNS_HARDENER
 Wire Wire Line
@@
 Connection ~ 13500 7200
 Wire Wire Line
-	13750 4150 13900 4150
-Wire Wire Line
 	13750 4550 13750 4450
 Wire Wire Line
@@
 	1    0    0    -1
 $EndComp
-Wire Wire Line
-	13900 4500 13900 4150
-Connection ~ 13900 4150
-Wire Wire Line
-	13900 4150 14350 4150
+Connection ~ 13900 4250
 $Comp
 L Device:LED_ALT D10
@@
 Wire Wire Line
 	14300 4700 14300 4750
+Wire Wire Line
+	13900 4500 13900 4250
+Wire Wire Line
+	13900 4250 14350 4250
+Wire Wire Line
+	13750 4150 14350 4150
+Text Notes 550  700  0    60   ~ 0
+84V When Charging
 $EndSCHEMATC

Commit message: Finalize layout for v0.0.15
Parts:
- removed PS1: TMR_6-7215WIR, Local:TRACO_TMR_6, symbol VDW_Modules:TMR_6-7215WIR
- added PS1: ERM01H110, VDW-Modules:ERM01H110, symbol VDW_Modules:ERM01H110
- added R25: 2.2k, Resistor_SMD:R_0805_2012Metric_Pad1.15x1.40mm_HandSolder, symbol Device:R_Small
- added R26: 4.7k, Resistor_SMD:R_0805_2012Metric_Pad1.15x1.40mm_HandSolder, symbol Device:R_Small
- PS2: footprint Local:RSDW20_H -> VDW-Modules:RSDW20_H
- U6: value HSCDLNN001PDAA3 -> HSCDANN005PGAA5; footprint Local:HoneyWell_LN -> VDW-Modules:HoneyWell_DIP_AN; Alt Vendor (none) -> Mouser; Alt Vendor P/N (none) -> 785-HSCDANN005PGAA5; MPN HSCDLNN001PDAA3 -> HSCDANN005PGAA5; Vendor P/N 480-5420-ND -> 480-6588-ND
Connections:
- wire segments 637 -> 643
- no-connect marks 36 -> 37
Other:
- note removed: "Temporarily SSCDRRN005PGAA5\nwith 2.2K and 4.7K voltage divider"
Changed lines of the file:
@@
 F 0 "PS2" H 4550 2237 60  0000 C CNN
 F 1 "RSDW20H-05" H 4550 2131 60  0000 C CNN
-F 2 "Local:RSDW20_H" H 4800 2200 60  0001 C CNN
+F 2 "VDW-Modules:RSDW20_H" H 4800 2200 60  0001 C CNN
 F 3 "http://www.meanwell.com/webapp/product/search.aspx?prod=RSDW20#1" H 4800 2200 60  0001 C CNN
 F 4 "~" H 850 250 50  0001 C CNN "Alt Vendor"
@@
 L power:+24V #PWR025
 U 1 1 5BBAFEC1
-P 5450 900
-F 0 "#PWR025" H 5450 750 50  0001 C CNN
-F 1 "+24V" H 5465 1073 50  0000 C CNN
-F 2 "" H 5450 900 50  0001 C CNN
-F 3 "" H 5450 900 50  0001 C CNN
-	1    5450 900
+P 5200 900
+F 0 "#PWR025" H 5200 750 50  0001 C CNN
+F 1 "+24V" H 5215 1073 50  0000 C CNN
+F 2 "" H 5200 900 50  0001 C CNN
+F 3 "" H 5200 900 50  0001 C CNN
+	1    5200 900
 	1    0    0    -1
 $EndComp
@@
 L power:GND #PWR012
 U 1 1 5BBEE83A
-P 5450 1200
-F 0 "#PWR012" H 5450 950 50  0001 C CNN
-F 1 "GND" H 5450 1050 50  0000 C CNN
-F 2 "" H 5450 1200 50  0001 C CNN
-F 3 "" H 5450 1200 50  0001 C CNN
-	1    5450 1200
+P 5050 1200
+F 0 "#PWR012" H 5050 950 50  0001 C CNN
+F 1 "GND" H 5050 1050 50  0000 C CNN
+F 2 "" H 5050 1200 50  0001 C CNN
+F 3 "" H 5050 1200 50  0001 C CNN
+	1    5050 1200
 	1    0    0    -1
 $EndComp
@@
 P 1450 8550
 F 0 "U6" H 1450 8987 60  0000 C CNN
-F 1 "HSCDLNN001PDAA3" H 1450 8881 60  0000 C CNN
-F 2 "Local:HoneyWell_LN" H 1450 8600 60  0001 C CNN
+F 1 "HSCDANN005PGAA5" H 1450 8881 60  0000 C CNN
+F 2 "VDW-Modules:HoneyWell_DIP_AN" H 1450 8600 60  0001 C CNN
 F 3 "https://sensing.honeywell.com/index.php?ci_id=151133" H 1450 8600 60  0001 C CNN
-F 4 "HSCDLNN001PDAA3" H 1450 8550 50  0001 C CNN "MPN"
+F 4 "HSCDANN005PGAA5" H 1450 8550 50  0001 C CNN "MPN"
 F 5 "DigiKey" H 1450 8550 50  0001 C CNN "Vendor"
-F 6 "480-5420-ND" H 1450 8550 50  0001 C CNN "Vendor P/N"
-F 7 "~" H -2250 2200 50  0001 C CNN "Alt Vendor"
-F 8 "~" H -2250 2200 50  0001 C CNN "Alt Vendor P/N"
+F 6 "480-6588-ND" H 1450 8550 50  0001 C CNN "Vendor P/N"
+F 7 "Mouser" H -2250 2200 50  0001 C CNN "Alt Vendor"
+F 8 "785-HSCDANN005PGAA5" H -2250 2200 50  0001 C CNN "Alt Vendor P/N"
 	1    1450 8550
 	-1   0    0    -1
@@
 	1850 8700 2000 8700
 Wire Wire Line
-	2000 8700 2000 9050
+	2000 8700 2000 9150
 Wire Wire Line
 	1850 8500 2000 8500
 Wire Wire Line
 	2000 8500 2000 8150
-$Comp
-L power:+3V3 #PWR032
-U 1 1 5BFAC91A
-P 2000 8150
-F 0 "#PWR032" H 2000 8000 50  0001 C CNN
-F 1 "+3V3" H 2000 8290 50  0000 C CNN
-F 2 "" H 2000 8150 50  0001 C CNN
-F 3 "" H 2000 8150 50  0001 C CNN
-	1    2000 8150
-	1    0    0    -1
-$EndComp
 Wire Wire Line
-	1850 8600 2500 8600
+	1850 8600 2150 8600
 $Comp
 L power:GND #PWR033
 U 1 1 5BFB5711
-P 2000 9050
-F 0 "#PWR033" H 2000 8800 50  0001 C CNN
-F 1 "GND" H 2000 8900 50  0000 C CNN
-F 2 "" H 2000 9050 50  0001 C CNN
-F 3 "" H 2000 9050 50  0001 C CNN
-	1    2000 9050
+P 2000 9200
+F 0 "#PWR033" H 2000 8950 50  0001 C CNN
+F 1 "GND" H 2000 9050 50  0000 C CNN
+F 2 "" H 2000 9200 50  0001 C CNN
+F 3 "" H 2000 9200 50  0001 C CNN
+	1    2000 9200
 	1    0    0    -1
 $EndComp
@@
 	-1   0    0    1
 $EndComp
-Text Label 2500 8600 2    60   ~ 0
+Text Label 2900 8850 2    60   ~ 0
 PRESS_SNS
 $Comp
@@
 Text Notes 1300 7400 0    60   ~ 0
 CABLE
-$Comp
-L VDW_Modules:TMR_6-7215WIR PS1
-U 1 1 5BC3AB94
-P 4650 1100
-F 0 "PS1" H 4600 1450 60  0000 C CNN
-F 1 "TMR_6-7215WIR" H 4650 1341 60  0000 C CNN
-F 2 "Local:TRACO_TMR_6" H 4350 1000 60  0001 C CNN
-F 3 "https://www.tracopower.com/products/tmr6wir.pdf" H 4350 1000 60  0001 C CNN
-F 4 "TMR_6-7215WIR" H 4650 1100 50  0001 C CNN "MPN"
-F 5 "DigiKey" H 4650 1100 50  0001 C CNN "Vendor"
-F 6 "1951-2035-ND" H 4650 1100 50  0001 C CNN "Vendor P/N"
-F 7 "~" H 200 0   50  0001 C CNN "Alt Vendor"
-F 8 "~" H 200 0   50  0001 C CNN "Alt Vendor P/N"
-	1    4650 1100
-	1    0    0    -1
-$EndComp
 Wire Wire Line
-	5200 1100 5450 1100
+	4900 1100 5050 1100
 Wire Wire Line
-	5450 1100 5450 1200
+	5050 1100 5050 1200
 Wire Wire Line
-	5200 1000 5450 1000
+	4900 1000 5200 1000
 Wire Wire Line
-	5450 1000 5450 900
+	5200 1000 5200 900
 Wire Wire Line
 	3900 900  3900 1000
@@
 Text Notes 800  5200 0    60   ~ 0
 KNOB: ML-75-1-6
-Text Notes 850  9000 0    60   ~ 0
-Temporarily SSCDRRN005PGAA5\nwith 2.2K and 4.7K voltage divider
 $Comp
 L Device:Thermistor TH1
@@
 L Device:R_Small R14
 U 1 1 5BEED4EC
-P 5600 1150
-F 0 "R14" V 5500 1150 50  0000 C CNN
-F 1 "7k" V 5600 1150 50  0000 C CNN
-F 2 "Resistor_SMD:R_0805_2012Metric_Pad1.15x1.40mm_HandSolder" H 5600 1150 50  0001 C CNN
-F 3 "~" H 5600 1150 50  0001 C CNN
-	1    5600 1150
+P 5400 1150
+F 0 "R14" V 5300 1150 50  0000 C CNN
+F 1 "7k" V 5400 1150 50  0000 C CNN
+F 2 "Resistor_SMD:R_0805_2012Metric_Pad1.15x1.40mm_HandSolder" H 5400 1150 50  0001 C CNN
+F 3 "~" H 5400 1150 50  0001 C CNN
+	1    5400 1150
 	-1   0    0    1
 $EndComp
@@
 L Device:LED_ALT D4
 U 1 1 5BEED62C
-P 5600 1450
-F 0 "D4" V 5638 1333 50  0000 R CNN
-F 1 "+24V" V 5547 1333 50  0000 R CNN
-F 2 "LED_SMD:LED_0805_2012Metric_Pad1.15x1.40mm_HandSolder" H 5600 1450 50  0001 C CNN
-F 3 "~" H 5600 1450 50  0001 C CNN
-	1    5600 1450
+P 5400 1450
+F 0 "D4" V 5438 1333 50  0000 R CNN
+F 1 "+24V" V 5347 1333 50  0000 R CNN
+F 2 "LED_SMD:LED_0805_2012Metric_Pad1.15x1.40mm_HandSolder" H 5400 1450 50  0001 C CNN
+F 3 "~" H 5400 1450 50  0001 C CNN
+	1    5400 1450
 	0    -1   -1   0
 $EndComp
-Connection ~ 5450 1000
+Connection ~ 5200 1000
 $Comp
 L power:GND #PWR0106
 U 1 1 5BF88E9D
-P 5600 1650
-F 0 "#PWR0106" H 5600 1400 50  0001 C CNN
-F 1 "GND" H 5600 1500 50  0000 C CNN
-F 2 "" H 5600 1650 50  0001 C CNN
-F 3 "" H 5600 1650 50  0001 C CNN
-	1    5600 1650
+P 5400 1650
+F 0 "#PWR0106" H 5400 1400 50  0001 C CNN
+F 1 "GND" H 5400 1500 50  0000 C CNN
+F 2 "" H 5400 1650 50  0001 C CNN
+F 3 "" H 5400 1650 50  0001 C CNN
+	1    5400 1650
 	1    0    0    -1
 $EndComp
@@
 	5200 2550 5200 2450
 Wire Wire Line
-	5600 1050 5600 1000
+	5400 1050 5400 1000
 Wire Wire Line
-	5450 1000 5600 1000
+	5200 1000 5400 1000
 Wire Wire Line
-	5600 1650 5600 1600
+	5400 1650 5400 1600
 Wire Wire Line
-	5600 1300 5600 1250
+	5400 1300 5400 1250
 $Comp
 L Device:R_Small R18
@@
 Text Notes 550  700  0    60   ~ 0
 84V When Charging
+$Comp
+L VDW_Modules:ERM01H110 PS1
+U 1 1 5C0BA996
+P 4500 1100
+F 0 "PS1" H 4500 1487 60  0000 C CNN
+F 1 "ERM01H110" H 4500 1381 60  0000 C CNN
+F 2 "VDW-Modules:ERM01H110" H 4500 1700 60  0001 C CNN
+F 3 "https://www.mouser.com/datasheet/2/633/erm20_ds_28mar2017_review_1491322745-1113377.pdf" H 4500 1800 60  0001 C CNN
+F 4 "ERM01H110" H 4500 1600 60  0001 C CNN "MPN"
+F 5 "Mouser" H 4500 2000 60  0001 C CNN "Vendor"
+F 6 "826-ERM01H110" H 4500 1900 60  0001 C CNN "Vendor P/N"
+	1    4500 1100
+	1    0    0    -1
+$EndComp
+NoConn ~ 4900 1200
+$Comp
+L Device:R_Small R25
+U 1 1 5C131D13
+P 2150 8700
+F 0 "R25" H 2209 8746 50  0000 L CNN
+F 1 "2.2k" H 2209 8655 50  0000 L CNN
+F 2 "Resistor_SMD:R_0805_2012Metric_Pad1.15x1.40mm_HandSolder" H 2150 8700 50  0001 C CNN
+F 3 "~" H 2150 8700 50  0001 C CNN
+	1    2150 8700
+	1    0    0    -1
+$EndComp
+$Comp
+L Device:R_Small R26
+U 1 1 5C132222
+P 2150 9000
+F 0 "R26" H 2209 9046 50  0000 L CNN
+F 1 "4.7k" H 2209 8955 50  0000 L CNN
+F 2 "Resistor_SMD:R_0805_2012Metric_Pad1.15x1.40mm_HandSolder" H 2150 9000 50  0001 C CNN
+F 3 "~" H 2150 9000 50  0001 C CNN
+	1    2150 9000
+	1    0    0    -1
+$EndComp
+Wire Wire Line
+	2150 8800 2150 8850
+Wire Wire Line
+	2150 9100 2150 9150
+Wire Wire Line
+	2150 9150 2000 9150
+Connection ~ 2000 9150
+Wire Wire Line
+	2000 9150 2000 9200
+Wire Wire Line
+	2150 8850 2900 8850
+Connection ~ 2150 8850
+Wire Wire Line
+	2150 8850 2150 8900
+$Comp
+L power:+5V #PWR0123
+U 1 1 5C37A782
+P 2000 8150
+F 0 "#PWR0123" H 2000 8000 50  0001 C CNN
+F 1 "+5V" H 2000 8290 50  0000 C CNN
+F 2 "" H 2000 8150 50  0001 C CNN
+F 3 "" H 2000 8150 50  0001 C CNN
+	1    2000 8150
+	1    0    0    -1
+$EndComp
 $EndSCHEMATC

Commit message: Change offboard component footprint from '~' to 'NoFootprint'
Parts:
- D1, J1, J10, J100, J102, J105, J12, J14, J3, J4, J5, J55, J6, J71, J8, J92, J93, J96, J98, J99, K1, LS1, R5, SP1, SP2, SP3, SP4, SP5, SP6, SP7, SW1, SW5, SW6, TH1, TH2, U10, U5, U9: footprint ~ -> NoFootprint:NoFootprint

Commit message: update footprints
Parts:
- J94: footprint Connector_Molex:Molex_SPOX_5267-02A_1x02_P2.50mm_Vertical -> VDW-Connectors:Molex-705430001_02x2.54mm_Straight
- U1: footprint Particle:photon_smd -> VDW-Particle:photon_smd
- U2: footprint Local:Adafruit_1096 -> VDW-Modules:SimpleRF_Receiver
- U3, U4: footprint Package_DIP:DIP-12_W10.16mm -> VDW-Modules:BOB-12_W10.16mm
Changed lines of the file:
@@
 F 0 "U3" H 13100 4797 60  0000 C CNN
 F 1 "BOB-12009" H 13100 4691 60  0000 C CNN
-F 2 "Package_DIP:DIP-12_W10.16mm" H 13800 4850 60  0001 C CNN
+F 2 "VDW-Modules:BOB-12_W10.16mm" H 13800 4850 60  0001 C CNN
 F 3 "https://www.sparkfun.com/products/12009" H 13800 4850 60  0001 C CNN
 F 4 "~" H 5000 500 50  0001 C CNN "Alt Vendor"
@@
 F 0 "U4" H 13100 7147 60  0000 C CNN
 F 1 "BOB-12009" H 13100 7041 60  0000 C CNN
-F 2 "Package_DIP:DIP-12_W10.16mm" H 13800 7200 60  0001 C CNN
+F 2 "VDW-Modules:BOB-12_W10.16mm" H 13800 7200 60  0001 C CNN
 F 3 "https://www.sparkfun.com/products/12009" H 13800 7200 60  0001 C CNN
 F 4 "~" H 5000 2850 50  0001 C CNN "Alt Vendor"
@@
 F 0 "U2" H 1156 6997 60  0000 C CNN
 F 1 "Adafruit_1096" H 1156 6891 60  0000 C CNN
-F 2 "Local:Adafruit_1096" H 2050 7050 60  0001 C CNN
+F 2 "VDW-Modules:SimpleRF_Receiver" H 2050 7050 60  0001 C CNN
 F 3 "https://www.adafruit.com/product/1096" H 2050 7050 60  0001 C CNN
 F 4 "Adafruit" H -1300 2450 50  0001 C CNN "Alt Vendor"
@@
 F 0 "J94" H 3300 1450 50  0000 C CNN
 F 1 "0705430001" H 3600 1150 50  0001 C CNN
-F 2 "Connector_Molex:Molex_SPOX_5267-02A_1x02_P2.50mm_Vertical" H 3200 1350 50  0001 C CNN
+F 2 "VDW-Connectors:Molex-705430001_02x2.54mm_Straight" H 3200 1350 50  0001 C CNN
 F 3 "https://www.molex.com/pdm_docs/sd/705430001_sd.pdf" H 3200 1350 50  0001 C CNN
 F 4 "0705430001" H 3200 1350 50  0001 C CNN "MPN"
@@
 F 0 "U1" H 9150 1878 50  0000 C CNN
 F 1 "Photon" H 9150 1787 50  0000 C CNN
-F 2 "Particle:photon_smd" H 9150 2700 50  0001 C CNN
+F 2 "VDW-Particle:photon_smd" H 9150 2700 50  0001 C CNN
 F 3 "https://media.digikey.com/pdf/Data%20Sheets/Particle%20PDFs/Photon_v015_Web.pdf" H 9150 2700 50  0001 C CNN
 F 4 "PHOTONNOH" H 9150 2700 50  0001 C CNN "MPN"
