File: PCB/MixController.kicad_pcb (KiCad board)
At the start: 2 copper layers, 150.2 x 127 mm, 174 parts, among them J101 B2B-PH-K-S(LF)(SN), J103 B3B-PH-K-S(LF)(SN), J104 B2B-XH-A(LF)(SN), J11 B5B-XH-A(LF)(SN), J13 B8B-XH-A(LF)(SN), J2 B2B-XH-A(LF)(SN), J38 B5B-PH-K-S(LF)(SN), J67 B6B-PH-K-S(LF)(SN), J7 B3B-XH-A(LF)(SN), J9 B2B-XH-A(LF)(SN)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

Commit message: update footprints
Parts:
- J94: footprint Connector_Molex:Molex_SPOX_5267-02A_1x02_P2.50mm_Vertical -> VDW-Connectors:Molex-705430001_02x2.54mm_Straight
- U1: footprint Particle:photon_smd -> VDW-Particle:photon_smd
- U2: footprint Local:Adafruit_1096 -> VDW-Modules:SimpleRF_Receiver
- U3, U4: footprint Package_DIP:DIP-12_W10.16mm -> VDW-Modules:BOB-12_W10.16mm
- moved U3 8.23 mm to (208.3, 56.4), turned to 0 degrees
- moved U4 8.23 mm to (104.2, 56.4), turned to 0 degrees
- moved J94 1.80 mm to (134.0, 34.9), turned to 0 degrees
Routing:
- net +72V: track 78.7 -> 77.4 mm
